File: hardware/FDC.sch (KiCad schematic (older format))
At the start: 2 parts, among them J2 Floppy, U1 FDC37C78

Commit message: FDC wiring
Parts:
- added C1: 0.1uF, Capacitor_SMD:C_0603_1608Metric_Pad1.08x0.95mm_HandSolder, symbol Device:CP1
- added J1: EXPANSION, Connector_PinHeader_2.54mm:PinHeader_2x20_P2.54mm_Vertical, symbol Connector_Generic:Conn_02x20_Odd_Even
- added X1: 24MHz, Oscillator:Oscillator_DIP-8, symbol Oscillator:CXO_DIP8
- added X2: CXO_DIP14, Oscillator:Oscillator_DIP-14, symbol Oscillator:CXO_DIP14
Connections:
- net +5V: now also C1.1, J1.1 (Pin_1), J1.2 (Pin_2), X1.8 (Vcc), X2.14 (Vcc)
- net CLK24: now also X1.5 (OUT), X2.8 (OUT)
- net CPU_A0: now also J1.21 (Pin_21)
- net CPU_A1: now also J1.23 (Pin_23)
- net CPU_A2: now also J1.25 (Pin_25)
- net CPU_D0: now also J1.22 (Pin_22)
- net CPU_D1: now also J1.24 (Pin_24)
- net CPU_D2: now also J1.26 (Pin_26)
- net CPU_D3: now also J1.28 (Pin_28)
- net CPU_D4: now also J1.30 (Pin_30)
- net CPU_D5: now also J1.32 (Pin_32)
- net CPU_D6: now also J1.34 (Pin_34)
- net CPU_D7: now also J1.36 (Pin_36)
- net FDC_RST: now also J1.8 (Pin_8)
- net GND: now also C1.2, J1.13 (Pin_13), J1.18 (Pin_18), J1.3 (Pin_3), J1.37 (Pin_37), J1.38 (Pin_38), J1.4 (Pin_4), J1.40 (Pin_40), X1.4 (GND), X2.7 (GND)
- net ~FDCSEL: now also J1.7 (Pin_7)
- net ~PRG_OE: now also J1.19 (Pin_19)
- net ~PRG_WE: now also J1.20 (Pin_20)
- net FDC_IRQ renamed ~IRQ
- net ~IRQ: now also J1.39 (Pin_39)
- new net CPU_A3: J1.27 (Pin_27)
- new net CPU_A4: J1.29 (Pin_29)
- new net CPU_A5: J1.31 (Pin_31)
- new net CPU_A6: J1.33 (Pin_33)
- new net CPU_A7: J1.35 (Pin_35)
- new net M2: J1.6 (Pin_6)
- new net SYSCLK: J1.5 (Pin_5)
- new net ~DEVSEL0: J1.10 (Pin_10)
- new net ~DEVSEL1: J1.11 (Pin_11)
- new net ~DEVSEL2: J1.16 (Pin_16)
- new net ~DEVSEL3: J1.15 (Pin_15)
- new net ~IOSEL0: J1.9 (Pin_9)
- new net ~IOSEL1: J1.12 (Pin_12)
- new net ~IOSEL2: J1.17 (Pin_17)
- new net ~IOSEL3: J1.14 (Pin_14)
