File: hardware/NESPC.kicad_pcb (KiCad board)
At the start: 4 copper layers, 120.4 x 92.7 mm, 21 parts, among them J1 NESCART, J2 Floppy, J3 EXPANSION, J6 JTAG, U1 FDC37C78, U2 CLONE CIC, U3 ATF1508, U5 512Kx8 SRAM PRG, U6 512Kx8 FLASH PRG, U7 512Kx8 SRAM CHR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

Commit message: FDC wiring
Parts:
- added J1: HOST, Connector_PinHeader_2.54mm:PinHeader_2x20_P2.54mm_Vertical, F.Cu at (207.0, 66.0)
- added X1: 24MHz, Oscillator:Oscillator_DIP-8, F.Cu at (217.2, 73.7)
- added X2: CXO_DIP14, Oscillator:Oscillator_DIP-14, F.Cu at (217.2, 73.7)
- C3: moved to F.Cu
- J2: value Floppy -> FLOPPY
- moved C4 116.4 mm to (157.5, 117.5), turned to 135 degrees
- moved C3 106.8 mm to (182.2, 142.0), turned to 270 degrees
- moved C2 93.9 mm to (173.4, 116.8), turned to 45 degrees
- moved C9 69.3 mm to (157.5, 126.4), turned to 135 degrees
- moved C1 66.8 mm to (217.8, 81.3)
- moved J2 54.2 mm to (242.6, 67.9)
- moved U1 48.0 mm to (224.8, 90.2), turned to 90 degrees
- renumbered J1 to J0
Connections:
- C1 pad 1: /+5V -> /FDC/+5V
- C1 pad 2: /GND -> /FDC/GND
- J3 pad 7: /GND -> /~FDCSEL
- J3 pad 8: /GND -> /FDC_RST
- U1 pad 13: /FDC/FDC_IRQ -> /FDC/~IRQ
- U3 pad 24: /~ROMSEL -> /~RAM_CE
- U3 pad 25: Net-(U3-Pad25) -> /~ROMSEL
- U3 pad 27: Net-(U3-Pad27) -> /CIRAM_A10
- U3 pad 28: Net-(U3-Pad28) -> /~FDCSEL
- U3 pad 29: Net-(U3-Pad29) -> /FDC_RST
- U3 pad 30: Net-(U3-Pad30) -> /CIRAM_~CE
Routing:
- net /CIRAM_A10: track 0.00 -> 130.3 mm
- net /CIRAM_~CE: track 0.00 -> 116.1 mm, vias 0 -> 1
- net /~RAM_CE: track 0.00 -> 95.8 mm, vias 0 -> 1
- net /~FDCSEL: track 0.00 -> 67.2 mm
- net /FDC/+5V: track 0.00 -> 61.0 mm, vias 0 -> 1
- net /FDC_RST: track 0.00 -> 60.9 mm
- net /FDC/~IRQ: track 0.00 -> 36.5 mm
- net /FDC/CLK24: track 0.00 -> 36.1 mm, vias 0 -> 1
- net /FDC/FLP_~DS0: track 0.00 -> 33.3 mm, vias 0 -> 2
- net /FDC/~FDCSEL: track 0.00 -> 29.8 mm, vias 0 -> 1
- net /FDC/FLP_~HDSEL: track 0.00 -> 29.3 mm, vias 0 -> 1
- net /FDC/FLP_DENSEL: track 0.00 -> 29.1 mm, vias 0 -> 1
- net /FDC/FLP_~WGATE: track 0.00 -> 28.4 mm
- net /FDC/FLP_~INDEX: track 0.00 -> 28.3 mm, vias 0 -> 1
- net /FDC/FLP_~DSKCHG: track 0.00 -> 28.3 mm, vias 0 -> 2
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- added copper zone on B.Cu, net /FDC/GND
- added copper zone on F.Cu, net /FDC/GND
Other:
- board size 120.4 x 92.7 mm -> 178.2 x 92.7 mm
