File: hardware/NESPC.kicad_pcb (KiCad board)
At the start: 4 copper layers, 165.7 x 100 mm, 33 parts, among them J0 NESCART, J1 HOST, J2 FLOPPY, J3 EXPANSION, J4 FLOPPY, J5 HOST, J6 JTAG, U1 FDC37C78, U2 CLONE CIC, U3 ATF1508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

Commit message: Finalized boards sent out for Rev.0
Parts:
- added Q1: 2N2222, Package_TO_SOT_THT:TO-92S_Wide, F.Cu at (231.7, 133.5)
- added Q2: 2N2222, Package_TO_SOT_THT:TO-92S_Wide, F.Cu at (233.2, 88.0)
- added R1: 1K, Resistor_SMD:R_0603_1608Metric_Pad0.98x0.95mm_HandSolder, F.Cu at (225.8, 131.0)
- added R2: 1K, Resistor_SMD:R_0603_1608Metric_Pad0.98x0.95mm_HandSolder, F.Cu at (231.7, 139.4)
- added R3: 1K, Resistor_SMD:R_0603_1608Metric_Pad0.98x0.95mm_HandSolder, B.Cu at (222.8, 87.0)
- added R4: 1K, Resistor_SMD:R_0603_1608Metric_Pad0.98x0.95mm_HandSolder, F.Cu at (232.2, 90.5)
Connections:
- J6 pad 2: /TMS -> /TDI
- J6 pad 3: /TCK -> /TMS
- J6 pad 5: /TDI -> /TCK
- U1 pad 13: /Floppy Disk Controller 37C78/~IRQ -> /Floppy Disk Controller 37C78/IRQ
- U1 pad 14: /Floppy Disk Controller 37C78/FDC_TC -> /Floppy Disk Controller 37C78/GND
- U1 pad 25: /Floppy Disk Controller 37C78/FLP_MEDIA_ID0 -> /Floppy Disk Controller 37C78/GND
- U1 pad 26: /Floppy Disk Controller 37C78/FLP_MEDIA_ID1 -> /Floppy Disk Controller 37C78/GND
- U4 pad 23: Net-(U4-Pad23) -> /Floppy Disk Controller 82077/IRQ
Routing:
- net /Floppy Disk Controller 37C78/~IRQ: track 29.3 -> 6.91 mm
- net /Floppy Disk Controller 37C78/IRQ: track 0.00 -> 12.8 mm
- net /Floppy Disk Controller 82077/IRQ: track 0.00 -> 11.6 mm, vias 0 -> 1
- net Net-(Q2-Pad2): track 0.00 -> 7.90 mm
- net /Floppy Disk Controller 82077/~IRQ: track 0.00 -> 6.74 mm
- net Net-(Q1-Pad2): track 0.00 -> 5.02 mm
- net Net-(Q1-Pad1): track 0.00 -> 5.00 mm
- net /Floppy Disk Controller 37C78/GND: track 16.6 -> 20.8 mm
- net Net-(Q2-Pad1): track 0.00 -> 2.54 mm
