File: hardware/NESPC.sch (KiCad schematic (older format))
At the start: 18 parts, among them J1 NESCART, J2 Floppy, J3 EXPANSION, J4 PPU Mirror X/Y, J5 PPU Nametable RAM, U1 ORIGINAL CIC, U10 512Kx8 FLASH PRG, U11 512Kx8 SRAM CHR, U12 512Kx8 FLASH CHR, U2 CLONE CIC, U3 WINDOW, U4 SLOT, U5 PRG MMU 0, U6 PRG MMU 1, U7 CHR MMU 0, U8 CHR MMU 1, U9 512Kx8 SRAM PRG, U9 FDC37C78

Commit message: CUPL Compliance
Connections:
- net +5V: no longer U5.23 (Pin_23), U7.23 (Pin_23), U8.23 (Pin_23)
- net CM0_LE: no longer U7.14 (Pin_14)
- net CM1_LE: no longer U8.14 (Pin_14)
- net GND: now also U5.14 (Pin_14), U5.2 (Pin_2), U5.23 (Pin_23), U6.14 (Pin_14), U7.14 (Pin_14), U7.2 (Pin_2), U7.23 (Pin_23), U8.14 (Pin_14), U8.2 (Pin_2), U8.23 (Pin_23); no longer U5.13 (Pin_13), U7.13 (Pin_13), U8.13 (Pin_13)
- net M2: now also U6.23 (Pin_23)
- net PM0_LE: no longer U5.14 (Pin_14)
- net PPU_A12: now also U7.13 (Pin_13); no longer U8.2 (Pin_2)
- net PPU_~A12: now also U8.13 (Pin_13); no longer U7.2 (Pin_2)
- net ~PAGEL: now also U5.13 (Pin_13); no longer U5.2 (Pin_2)
- no-connect marks 13 -> 11
Changed lines of the file:
@@
 Text Label 9000 4500 0    50   ~ 0
 PMU_A15
-Text Label 9000 2700 0    50   ~ 0
+Text Label 8500 3700 2    50   ~ 0
 PPU_A12
 Wire Wire Line
-	9000 2700 9750 2700
+	8500 3700 7750 3700
 Wire Wire Line
 	10250 4700 11000 4700
@@
 Text Label 3500 3500 2    50   ~ 0
 MMU_A19
-Wire Wire Line
-	2750 2700 3500 2700
-Text Label 3500 2700 2    50   ~ 0
-+5V
-Wire Wire Line
-	2750 3600 3500 3600
-Text Label 3500 3600 2    50   ~ 0
-PM0_LE
 $Comp
 L Connector_Generic:Conn_02x12_Counter_Clockwise U7
@@
 Text Label 6500 3100 0    50   ~ 0
 CPU_D3
-Wire Wire Line
-	6500 3600 7250 3600
-Text Label 6500 3600 0    50   ~ 0
-GND
-Wire Wire Line
-	7750 2700 8500 2700
-Text Label 8500 2700 2    50   ~ 0
-+5V
-Wire Wire Line
-	7750 3600 8500 3600
-Text Label 8500 3600 2    50   ~ 0
-CM0_LE
 $Comp
 L Connector_Generic:Conn_02x12_Counter_Clockwise U8
@@
 Text Label 9000 3600 0    50   ~ 0
 GND
-Wire Wire Line
-	10250 2700 11000 2700
-Text Label 11000 2700 2    50   ~ 0
-+5V
-Wire Wire Line
-	10250 3600 11000 3600
-Text Label 11000 3600 2    50   ~ 0
-CM1_LE
-Text Label 6500 2700 0    50   ~ 0
+Text Label 11000 3700 2    50   ~ 0
 PPU_~A12
 Wire Wire Line
-	6500 2700 7250 2700
+	11000 3700 10250 3700
 Wire Wire Line
 	10250 3400 11000 3400
@@
 ~PAGEL
 Wire Wire Line
-	2250 2700 1500 2700
-Text Label 1500 2700 0    50   ~ 0
+	2750 3700 3500 3700
+Text Label 3500 3700 2    50   ~ 0
 ~PAGEL
-Wire Wire Line
-	1500 3600 2250 3600
-Text Label 1500 3600 0    50   ~ 0
-GND
 Wire Wire Line
 	6500 3700 7250 3700
@@
 	9000 3700 9750 3700
 Text Label 9000 3700 0    50   ~ 0
-GND
-Wire Wire Line
-	8500 3700 7750 3700
-Text Label 8500 3700 2    50   ~ 0
 GND
 Wire Wire Line
@@
 Text Label 3500 2600 2    50   ~ 0
 +5V
-Text Label 3500 3700 2    50   ~ 0
-GND
-Wire Wire Line
-	3500 3700 2750 3700
 $Comp
 L Connector_Generic:Conn_02x12_Counter_Clockwise U6
@@
 Text Label 4000 3000 0    50   ~ 0
 CPU_A14
-Wire Wire Line
-	4000 2700 4750 2700
-Text Label 4000 2700 0    50   ~ 0
-~ROMSEL
 Wire Wire Line
 	4000 6600 4750 6600
@@
 	1    0    0    -1
 $EndComp
-Wire Wire Line
-	11000 3700 10250 3700
-Text Label 11000 3700 2    50   ~ 0
-GND
-Wire Wire Line
-	6000 3700 5250 3700
-Text Label 6000 3700 2    50   ~ 0
-GND
 Text Label 6000 3500 2    50   ~ 0
 MMU_A19
@@
 Wire Wire Line
 	5250 3400 6000 3400
-NoConn ~ 5250 2700
-NoConn ~ 5250 3600
 Wire Wire Line
 	9000 6600 9750 6600
@@
 Text Label 1500 1700 0    50   ~ 0
 CPU_A2
+Text Label 4000 2700 0    50   ~ 0
+~ROMSEL
+Wire Wire Line
+	4000 2700 4750 2700
+Text Label 1500 3600 0    50   ~ 0
+GND
+Wire Wire Line
+	1500 3600 2250 3600
+Text Label 1500 2700 0    50   ~ 0
+GND
+Wire Wire Line
+	1500 2700 2250 2700
+Text Label 6000 3700 2    50   ~ 0
+GND
+Wire Wire Line
+	6000 3700 5250 3700
+Wire Wire Line
+	6000 2700 5250 2700
+Text Label 6000 2700 2    50   ~ 0
+M2
+Text Label 3500 2700 2    50   ~ 0
+GND
+Wire Wire Line
+	3500 2700 2750 2700
+Text Label 6000 3600 2    50   ~ 0
+GND
+Wire Wire Line
+	6000 3600 5250 3600
+Text Label 3500 3600 2    50   ~ 0
+GND
+Wire Wire Line
+	3500 3600 2750 3600
+Text Label 6500 3600 0    50   ~ 0
+GND
+Wire Wire Line
+	6500 3600 7250 3600
+Text Label 6500 2700 0    50   ~ 0
+GND
+Wire Wire Line
+	6500 2700 7250 2700
+Text Label 9000 2700 0    50   ~ 0
+GND
+Wire Wire Line
+	9000 2700 9750 2700
+Text Label 11000 2700 2    50   ~ 0
+GND
+Wire Wire Line
+	11000 2700 10250 2700
+Text Label 11000 3600 2    50   ~ 0
+GND
+Wire Wire Line
+	11000 3600 10250 3600
+Text Label 8500 3600 2    50   ~ 0
+GND
+Wire Wire Line
+	8500 3600 7750 3600
+Text Label 8500 2700 2    50   ~ 0
+GND
+Wire Wire Line
+	8500 2700 7750 2700
 $EndSCHEMATC

Commit message: PCB for ATF1508 Based Cart
Parts:
- removed J2: Floppy, symbol Connector_Generic:Conn_02x17_Odd_Even
- removed J4: PPU Mirror X/Y, symbol Connector_Generic:Conn_01x03
- removed J5: PPU Nametable RAM, symbol Connector_Generic:Conn_01x03
- removed U1: ORIGINAL CIC, symbol Connector_Generic:Conn_02x08_Counter_Clockwise
- removed U3: WINDOW, symbol Connector_Generic:Conn_02x12_Counter_Clockwise
- removed U4: SLOT, symbol Connector_Generic:Conn_02x12_Counter_Clockwise
- removed U5: PRG MMU 0, symbol Connector_Generic:Conn_02x12_Counter_Clockwise
- removed U6: PRG MMU 1, symbol Connector_Generic:Conn_02x12_Counter_Clockwise
- removed U7: CHR MMU 0, symbol Connector_Generic:Conn_02x12_Counter_Clockwise
- removed U8: CHR MMU 1, symbol Connector_Generic:Conn_02x12_Counter_Clockwise
- removed U9: FDC37C78, symbol Connector_Generic:Conn_02x24_Counter_Clockwise
- added C1, C10, C2, C3, C4, C5, C6, C7, C8, C9: 0.1uF, Capacitor_SMD:C_0603_1608Metric_Pad1.08x0.95mm_HandSolder, symbol Device:CP1
- added J6: JTAG, Connector_PinHeader_2.54mm:PinHeader_1x06_P2.54mm_Vertical, symbol Connector_Generic:Conn_01x06
- added U3: ATF1508, Package_LCC:PLCC-84, symbol atf1508:ATF1508
- J1: footprint (none) -> nes:NES_CART
- J3: footprint (none) -> Connector_PinHeader_2.54mm:PinHeader_2x20_P2.54mm_Vertical
- U2: footprint (none) -> Package_DIP:DIP-8_W7.62mm
- U5: renamed from U9; footprint (none) -> Package_DIP:DIP-32_W15.24mm
- U6: renamed from U10; footprint (none) -> Package_DIP:DIP-32_W15.24mm
- U7: renamed from U11; footprint (none) -> Package_DIP:DIP-32_W15.24mm
- U8: renamed from U12; footprint (none) -> Package_DIP:DIP-32_W15.24mm
Connections:
- net +5V: now also C1.1, C10.1, C2.1, C3.1, C4.1, C5.1, C6.1, C7.1, C8.1, C9.1, J6.1 (Pin_1), U3.13 (VCC), U3.26 (VCC), U3.3 (VCC), U3.38 (VCC), U3.43 (VCC), U3.53 (VCC), U3.66 (VCC), U3.78 (VCC)
- net CIRAM_A10: now also U3.29 (I/O)
- net CIRAM_~CE: now also U3.30 (I/O)
- net CPU_A0: now also U3.51 (I/O)
- net CPU_A1: now also U3.54 (I/O)
- net CPU_A10: now also U3.6 (I/O)
- net CPU_A11: now also U3.4 (I/O)
- net CPU_A12: now also U3.74 (I/O)
- net CPU_A13: now also U3.73 (I/O)
- net CPU_A14: now also U3.70 (I/O)
- net CPU_A2: now also U3.56 (I/O)
- net CPU_A3: now also U3.58 (I/O)
- net CPU_A4: now also U3.61 (I/O)
- net CPU_A5: now also U3.64 (I/O)
- net CPU_A6: now also U3.67 (I/O)
- net CPU_A7: now also U3.69 (I/O)
- net CPU_A8: now also U3.79 (I/O)
- net CPU_A9: now also U3.80 (I/O)
- net CPU_D0: now also U3.52 (I/O)
- net CPU_D1: now also U3.50 (I/O)
- net CPU_D2: now also U3.55 (I/O)
- net CPU_D3: now also U3.57 (I/O)
- net CPU_D4: now also U3.60 (I/O)
- net CPU_D5: now also U3.63 (I/O)
- net CPU_D6: now also U3.65 (I/O)
- net CPU_D7: now also U3.68 (I/O)
- net CPU_R~W: now also U3.31 (I/O)
- net FDC_RST: now also U3.27 (I/O)
- net GND: now also C1.2, C10.2, C2.2, C3.2, C4.2, C5.2, C6.2, C7.2, C8.2, C9.2, J6.6 (Pin_6), U3.19 (GND), U3.32 (GND), U3.42 (GND), U3.47 (GND), U3.59 (GND), U3.7 (GND), U3.72 (GND), U3.82 (GND)
- net M2: now also U3.81 (I/O/GCK3)
- net MMU_A12: now also U3.11 (I/O)
- net MMU_A13: now also U3.77 (I/O)
- net MMU_A14: now also U3.76 (I/O)
- net MMU_A15: now also U3.12 (I/O/PD1)
- net MMU_A16: now also U3.10 (I/O)
- net MMU_A17: now also U3.75 (I/O)
- net MMU_A18: now also U3.9 (I/O)
- net PMU_A12: now also U3.21 (I/O)
- net PMU_A13: now also U3.22 (I/O)
- net PMU_A14: now also U3.20 (I/O)
- net PMU_A15: now also U3.18 (I/O)
- net PMU_A16: now also U3.16 (I/O)
- net PMU_A17: now also U3.17 (I/O)
- net PMU_A18: now also U3.15 (I/O)
- net PPU_A10: now also J1.63 (Pin_63); no longer J1.62 (Pin_62)
- net PPU_A11: now also J1.62 (Pin_62); no longer J1.63 (Pin_63)
- net PPU_A12: now also U3.34 (I/O)
- net PPU_A13: now also U3.33 (I/O/TDI); no longer U7.22 (Pin_22), U8.22 (Pin_22)
- net SYSCLK: now also U3.83 (IINPUT/GCLK1)
- net ~DEVSEL0: now also U3.37 (I/O)
- net ~DEVSEL1: now also U3.41 (I/O)
- net ~DEVSEL2: now also U3.45 (I/O/PD2)
- net ~DEVSEL3: now also U3.46 (I/O)
- net ~FDCSEL: now also U3.28 (I/O/PD2)
- net ~IOSEL0: now also U3.39 (I/O/TMS)
- net ~IOSEL1: now also U3.40 (I/O)
- net ~IOSEL2: now also U3.48 (I/O)
- net ~IOSEL3: now also U3.44 (I/O)
- net ~PRG_OE: now also U3.5 (I/O)
- net ~PRG_WE: now also U3.49 (I/O)
- net ~RAM_CE: now also U3.24 (I/O)
- net ~ROMSEL: now also U3.25 (I/O)
- net ~ROM_CE: now also U3.8 (I/O)
- new net TCK: J6.3 (Pin_3), U3.62 (I/O/TCK)
- new net TDI: J6.5 (Pin_5), U3.14 (I/O/TDI)
- new net TDO: J6.4 (Pin_4), U3.71 (I/O/TDO)
- new net TMS: J6.2 (Pin_2), U3.23 (I/O/TMS)
- new net ~CHR_RAM_CE: U3.36 (I/O/PD1), U7.22 (Pin_22)
- new net ~CHR_ROM_CE: U3.35 (I/O), U8.22 (Pin_22)
- no-connect marks 11 -> 2
Other:
- moved on the sheet: J1, U5, U6, U7, U8

Commit message: FDC wiring
Parts:
- removed C1: 0.1uF, Capacitor_SMD:C_0603_1608Metric_Pad1.08x0.95mm_HandSolder, symbol Device:CP1
- renumbered J1 to J0
Connections:
- net CIRAM_A10: now also U3.27 (I/O); no longer U3.29 (I/O)
- net FDC_RST: now also J3.8 (Pin_8), U3.29 (I/O); no longer U3.27 (I/O)
- net GND: no longer J3.7 (Pin_7), J3.8 (Pin_8)
- net ~FDCSEL: now also J3.7 (Pin_7)
Changed lines of the file:
@@
 $EndDescr
 $Comp
-L Connector_Generic:Conn_02x36_Top_Bottom J1
+L Connector_Generic:Conn_02x36_Top_Bottom J0
 U 1 1 6348C45D
 P 15200 2550
-F 0 "J1" H 15250 4467 50  0000 C CNN
+F 0 "J0" H 15250 4467 50  0000 C CNN
 F 1 "NESCART" H 15250 4376 50  0000 C CNN
 F 2 "nes:NES_CART" H 15200 2550 50  0001 C CNN
@@
 M2
 Wire Wire Line
-	14000 7400 14750 7400
-Text Label 14000 7400 0    50   ~ 0
-GND
-Wire Wire Line
 	16000 7200 15250 7200
 Text Label 16000 7200 2    50   ~ 0
@@
 PPU_D4
 Wire Wire Line
-	7000 8550 6250 8550
-Text Label 6250 8550 0    50   ~ 0
+	7000 8350 6250 8350
+Text Label 6250 8350 0    50   ~ 0
 CIRAM_A10
 Wire Wire Line
@@
 	16000 7900 15250 7900
 Text Label 16000 7900 2    50   ~ 0
-GND
-Wire Wire Line
-	16000 7400 15250 7400
-Text Label 16000 7400 2    50   ~ 0
 GND
 Wire Wire Line
@@
 CIRAM_~CE
 Wire Wire Line
-	7000 8350 6250 8350
-Text Label 6250 8350 0    50   ~ 0
+	7000 8550 6250 8550
+Text Label 6250 8550 0    50   ~ 0
 FDC_RST
 Wire Wire Line
@@
 TDO
 $Comp
-L Device:CP1 C1
-U 1 1 6ED7805E
-P 2200 6500
-F 0 "C1" H 2315 6546 50  0000 L CNN
-F 1 "0.1uF" H 2315 6455 50  0000 L CNN
-F 2 "Capacitor_SMD:C_0603_1608Metric_Pad1.08x0.95mm_HandSolder" H 2200 6500 50  0001 C CNN
-F 3 "~" H 2200 6500 50  0001 C CNN
-	1    2200 6500
-	1    0    0    -1
-$EndComp
-$Comp
 L Device:CP1 C2
 U 1 1 6EDE0374
@@
 $EndComp
 Wire Wire Line
-	2200 6350 2200 6050
-Wire Wire Line
-	2200 6050 2650 6050
-Wire Wire Line
 	4000 6050 4000 6350
 Wire Wire Line
@@
 	4000 6950 3550 6950
 Wire Wire Line
-	2200 6950 2200 6650
-Wire Wire Line
 	2650 6650 2650 6950
 Connection ~ 2650 6950
 Wire Wire Line
-	2650 6950 2200 6950
-Wire Wire Line
 	3100 6650 3100 6950
 Connection ~ 3100 6950
@@
 Wire Wire Line
 	3550 6950 3100 6950
-Wire Wire Line
-	1450 6050 2200 6050
 Text Label 1450 6050 0    50   ~ 0
 +5V
 Text Label 1450 6950 0    50   ~ 0
 GND
-Wire Wire Line
-	1450 6950 2200 6950
-Connection ~ 2200 6950
-Connection ~ 2200 6050
 $Comp
 L Device:CP1 C6
@@
 F1 "FDC.sch" 50
 $EndSheet
+Wire Wire Line
+	14000 7400 14750 7400
+Text Label 14000 7400 0    50   ~ 0
+~FDCSEL
+Wire Wire Line
+	15250 7400 16000 7400
+Text Label 16000 7400 2    50   ~ 0
+FDC_RST
+Wire Wire Line
+	1450 6050 2650 6050
+Wire Wire Line
+	1450 6950 2650 6950
 $EndSCHEMATC

Commit message: Update NESPC.sch
Changed lines of the file:
@@
 $EndComp
-Wire Wire Line
-	12150 7350 11400 7350
-Text Label 11400 7350 0    50   ~ 0
-FDC_TC
-Wire Wire Line
-	12150 7750 11400 7750
-Text Label 11400 7750 0    50   ~ 0
-FLP_DRVDEN0
-Wire Wire Line
-	12150 7850 11400 7850
-Text Label 11400 7850 0    50   ~ 0
-FLP_DRVDEN1
-Wire Wire Line
-	12700 7900 13450 7900
-Text Label 13450 7900 2    50   ~ 0
-FLP_MEDIA_ID0
-Wire Wire Line
-	12700 7800 13450 7800
-Text Label 13450 7800 2    50   ~ 0
-FLP_MEDIA_ID1
-Wire Wire Line
-	12150 7250 11400 7250
-Text Label 11400 7250 0    50   ~ 0
-FDC_IRQ
 Wire Wire Line
 	6000 3500 5250 3500
@@
 CPU_A7
 $Sheet
-S 21600 700  11000 9900
+S 14500 5000 1150 400
 U 75E32237
-F0 "FDC" 50
+F0 "Floppy Disk Controller" 50
 F1 "FDC.sch" 50
 $EndSheet
