File: hardware/NESPC-FDC82077.kicad_pcb (KiCad board)
At the start: 4 copper layers, 165.7 x 100 mm, 33 parts, among them J0 NESCART, J1 HOST, J2 FLOPPY, J3 EXPANSION, J4 FLOPPY, J5 HOST, J6 JTAG, U1 FDC37C78, U2 CLONE CIC, U3 ATF1508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

Commit message: Finalized boards sent out for Rev.0
Parts:
- removed C1, C10, C2, C3, C4, C5, C6, C7, C8, C9: 0.1uF, Capacitor_SMD:C_0603_1608Metric_Pad1.08x0.95mm_HandSolder
- removed J0: NESCART, nes:NES_CART
- removed J1: HOST, Connector_PinHeader_2.54mm:PinHeader_2x20_P2.54mm_Vertical
- removed J2: FLOPPY, Connector_PinHeader_2.54mm:PinHeader_2x17_P2.54mm_Vertical
- removed J3: EXPANSION, Connector_PinHeader_2.54mm:PinHeader_2x20_P2.54mm_Vertical
- removed J6: JTAG, Connector_PinHeader_2.54mm:PinHeader_1x06_P2.54mm_Vertical
- removed U1: FDC37C78, Package_QFP:LQFP-48_7x7mm_P0.5mm
- removed U2: CLONE CIC, Package_DIP:DIP-8_W7.62mm
- removed U3: ATF1508, Package_LCC:PLCC-84
- removed U5: 512Kx8 SRAM PRG, Package_DIP:DIP-32_W15.24mm
- removed U6: 512Kx8 FLASH PRG, Package_DIP:DIP-32_W15.24mm
- removed U7: 512Kx8 SRAM CHR, Package_DIP:DIP-32_W15.24mm
- removed U8: 512Kx8 FLASH CHR, Package_DIP:DIP-32_W15.24mm
- removed X1: 24MHz, Oscillator:Oscillator_DIP-8
- removed X2: CXO_DIP14, Oscillator:Oscillator_DIP-14
- added Q2: 2N2222, Package_TO_SOT_THT:TO-92S_Wide, F.Cu at (233.2, 87.6)
- added R3: 1K, Resistor_SMD:R_0603_1608Metric_Pad0.98x0.95mm_HandSolder, B.Cu at (222.8, 87.0)
- added R4: 1K, Resistor_SMD:R_0603_1608Metric_Pad0.98x0.95mm_HandSolder, F.Cu at (232.2, 90.5)
Connections:
- U4 pad 23: Net-(U4-Pad23) -> /Floppy Disk Controller 82077/IRQ
Routing:
- net /+5V: track 449.6 -> 0.00 mm, vias 11 -> 0
- net /CPU_A7: track 177.3 -> 0.00 mm, vias 2 -> 0
- net /CPU_A2: track 175.6 -> 0.00 mm, vias 2 -> 0
- net /CPU_A6: track 174.8 -> 0.00 mm, vias 2 -> 0
- net /CPU_A3: track 172.8 -> 0.00 mm, vias 2 -> 0
- net /CPU_A5: track 172.4 -> 0.00 mm, vias 2 -> 0
- net /CPU_A4: track 171.3 -> 0.00 mm, vias 2 -> 0
- net /CPU_A1: track 170.4 -> 0.00 mm, vias 1 -> 0
- net /CPU_A11: track 166.9 -> 0.00 mm, vias 4 -> 0
- net /CPU_A0: track 165.3 -> 0.00 mm, vias 1 -> 0
- net /CPU_D0: track 164.3 -> 0.00 mm, vias 1 -> 0
- net /CPU_D7: track 163.5 -> 0.00 mm, vias 1 -> 0
- net /CPU_D2: track 162.9 -> 0.00 mm, vias 1 -> 0
- net /CPU_D1: track 162.6 -> 0.00 mm, vias 1 -> 0
- net /CPU_D3: track 162.3 -> 0.00 mm, vias 1 -> 0
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- removed copper zone on B.Cu, net /Floppy Disk Controller 37C78/GND
- removed copper zone on F.Cu, net /Floppy Disk Controller 37C78/GND
- removed copper zone on B.Cu, net /GND
- removed copper zone on F.Cu, net /GND
Other:
- board size 165.7 x 100 mm -> 55.2 x 49.5 mm
- board text removed: "GND"
- board text removed: "TCK"
- board text removed: "TDI"
- board text removed: "TDO"
- board text removed: "TMS"
- board text removed: "VCC"
